File: nms-210.kicad_pcb (KiCad board)
At the start: 2 copper layers, 77.2 x 129.5 mm, 12 parts, among them J1 Conn_02x25_Counter_Clockwise, U1 74LS138, U10 74LS240, U11 74LS240, U2 74LS138, U3 74LS74, U4 74LS08, U5 74LS175, U6 74LS373, U7 74LS04, U8 74LS240, U9 7438

Commit message: Sync latest status
Parts:
- added Con1: MSX_CARTRIDGE_PCB, Library:msx_cartridge, F.Cu at (198.4, 153.1)
- moved U11 193.8 mm to (230.1, 46.5), turned to -90 degrees
- moved U1 177.7 mm to (231.1, 124.0), turned to -90 degrees
- moved U9 176.6 mm to (229.9, 62.0), turned to -90 degrees
- moved U3 166.9 mm to (229.9, 108.2), turned to -90 degrees
- moved U7 166.4 mm to (229.6, 78.0), turned to -90 degrees
- moved U5 165.1 mm to (230.6, 93.5), turned to -90 degrees
- moved J1 133.8 mm to (170.2, 25.9), turned to 90 degrees
- moved U2 119.1 mm to (197.9, 124.0), turned to -90 degrees
- moved U10 117.9 mm to (196.6, 61.5), turned to -90 degrees
- moved U4 102.7 mm to (196.6, 108.2), turned to -90 degrees
- moved U8 102.6 mm to (196.8, 77.7), turned to -90 degrees
- moved U6 99.1 mm to (197.4, 93.5), turned to -90 degrees
Other:
- board size 77.2 x 129.5 mm -> 99.1 x 64 mm
