File: nms-210.kicad_sch (KiCad schematic)
At the start: 12 parts, among them J1 Conn_02x25_Counter_Clockwise, U1 74LS138, U10 74LS240, U11 74LS240, U2 74LS138, U3 74LS74, U4 74LS08, U5 74LS175, U6 74LS373, U7 74LS04, U8 74LS240, U9 7438

Commit message: Sync latest status
Parts:
- added Con1: MSX_CARTRIDGE_PCB, Library:msx_cartridge, symbol v9958:MSX_CARTRIDGE_PCB
Connections:
- no-connect marks 0 -> 2
Other:
- moved on the sheet: J1, U10, U11, U3A, U3B, U3C, U5, U6, U8, U9A, U9B, U9C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
